File: AuralFocus/hardware/aurial1/aurialPiHat/aurialPiHat.kicad_sch (KiCad schematic)
At the start: 13 parts, among them J1 GPIO, U1 CAT24C256, U2 STM32H753VITx

Commit message: Microfones e reguladores para os microfones
Parts:
- removed MK1, MK2, MK3, MK4, MK5, MK6: IM69D130, Sensor_Audio:Infineon_PG-LLGA-5-1, symbol Sensor_Audio:IM69D130
- added C19, C20, C21, C22, C23, C24: 100 ηF, symbol Device:C_Small
- added C25, C26, C27, C28: 1μF X7R 10V, symbol Device:C_Small
- added D1: APA102-2020, LED_SMD:LED-APA102-2020, symbol LED:APA102-2020
- added FB1, FB2: 600 Ω SMD, symbol Device:FerriteBead_Small
- added J2: Conn_Mic_Left_1, symbol Connector:Conn_01x05_Pin
- added J3: Conn_Mic_Left_2, symbol Connector:Conn_01x05_Pin
- added J4: Conn_Mic_Left_3, symbol Connector:Conn_01x05_Pin
- added J5: Conn_Mic_Right_1, symbol Connector:Conn_01x05_Pin
- added J6: Conn_Mic_Right_2, symbol Connector:Conn_01x05_Pin
- added J7: Conn_Mic_Right_3, symbol Connector:Conn_01x05_Pin
- added SW1: SW_MEC_5G, Button_Switch_SMD:SW_MEC_5GSH9, symbol Switch:SW_MEC_5G
- added U3: TPS7A4700RGWR, TPS7A4700RGWR:QFN65P500X500X100-21N, symbol TPS7A4700:TPS7A4700RGWR
- added U4, U6: TPS7A2033DQN, Package_SON:Texas_X2SON-4_1x1mm_P0.65mm, symbol Regulator_Linear:TPS7A20xxxDQN
Connections:
- net +5V: now also FB1.2, FB2.2
- net GND: now also C19.2, C20.2, C21.2, C22.2, C23.2, C24.2, C25.2, C26.2, C27.2, C28.2, J2.2 (Pin_2), J2.5 (Pin_5), J3.2 (Pin_2), J3.5 (Pin_5), J4.2 (Pin_2), J4.5 (Pin_5), J5.2 (Pin_2), J6.2 (Pin_2), J7.2 (Pin_2), U4.2 (GND), U6.2 (GND)
- net EN LEFT: now reaches U2.37 (PE7)
- net EN LEFT: now also U4.3 (EN)
- net EN RIGHT: now reaches U2.38 (PE8)
- net EN RIGHT: now also U6.3 (EN)
- new net: C25.1, FB1.1, U4.4 (IN)
- new net: U3.1 (OUT), U3.20 (OUT)
- new net: U3.15 (IN), U3.16 (IN)
- new net: C27.1, FB2.1, U6.4 (IN)
- new net: SW1.1 (A), SW1.2 (A)
- new net: SW1.3 (B), SW1.4 (B)
- new net PDM_CLOCK: J2.3 (Pin_3), J3.3 (Pin_3), J4.3 (Pin_3), J5.3 (Pin_3), J6.3 (Pin_3), J7.3 (Pin_3)
- new net PDM_DATA0: J2.4 (Pin_4), J5.4 (Pin_4)
- new net PDM_DATA1: J3.4 (Pin_4), J6.4 (Pin_4)
- new net PDM_DATA2: J4.4 (Pin_4), J7.4 (Pin_4)
- new net VDD LEFT 3.3: C19.1, C20.1, C21.1, C26.1, J2.1 (Pin_1), J3.1 (Pin_1), J4.1 (Pin_1), U4.1 (OUT)
- new net VDD RIGHT 3.3: C22.1, C23.1, C24.1, C28.1, J5.1 (Pin_1), J5.5 (Pin_5), J6.1 (Pin_1), J6.5 (Pin_5), J7.1 (Pin_1), J7.5 (Pin_5), U6.1 (OUT)
Other:
- added sheet Mic_Left_1 (mics.kicad_sch)
- added sheet Mic_Left_2 (mics.kicad_sch)
- added sheet Mic_Left_3 (mics.kicad_sch)
- added sheet Mic_Right_1 (mics.kicad_sch)
- added sheet Mic_Right_2 (mics.kicad_sch)
- added sheet Mic_Roght_3 (mics.kicad_sch)
- moved on the sheet: C1, JP1, R1, R2, U1

Commit message: Correções no filtro do regulador de 3.3V
Parts:
- removed C1: 100n, symbol Device:C_Small
- removed C27: 1μF X7R 10V, symbol Device:C_Small
- removed R1, R2: 3.9k, symbol Device:R_Small
- removed U6: TPS7A2033DQN, Package_SON:Texas_X2SON-4_1x1mm_P0.65mm, symbol Regulator_Linear:TPS7A20xxxDQN
- added C27, C29: 10μF, symbol Device:C_Polarized
- added C30, C31: 100ηF, symbol Device:C_Small
- added C32: 2.2μF X7R 10V, symbol Device:C_Small
- added C33: 100n, symbol Device:C_Small
- added R13, R14: 3.9k, symbol Device:R_Small
- added U5: TPS7A2033DQN, Package_SON:Texas_X2SON-4_1x1mm_P0.65mm, symbol Regulator_Linear:TPS7A20xxxDQN
- C25, C28: value 1μF X7R 10V -> 1μF; Tensão (none) -> 10V; Tipo (none) -> X7R
- C26: value 1μF X7R 10V -> 2.2μF X7R 10V; Encapsulamento (none) -> 0805/0603
Connections:
- net +3V3: now also C33.1, R13.1, R14.1
- net GND: now also U4.5 (Pad), C27.2, C29.2, C30.2, C31.2, C32.2, C33.2, U5.2 (GND), U5.5 (Pad)
- net ID_SCL: now also R14.2
- net ID_SDA: now also R13.2
- net VDD RIGHT 3.3: no longer C22.1, C23.1, C24.1, C28.1, J5.1 (Pin_1), J6.1 (Pin_1), J6.5 (Pin_5), J7.1 (Pin_1), J7.5 (Pin_5)
- net at C25.1, FB1.1, U4.4 (IN): now also C29.1, C31.1
- net at FB2.1: now also C28.1, C27.1, C30.1, U5.4 (IN)
- net EN LEFT renamed EN_LEFT
- net EN_LEFT: now also U5.3 (EN)
- net EN RIGHT renamed EN_RIGHT
- net VDD LEFT 3.3 renamed VDD_LEFT_3.3
- new net VDD_RIGHT_3.3: C22.1, C23.1, C24.1, C32.1, J5.1 (Pin_1), J6.1 (Pin_1), J6.5 (Pin_5), J7.1 (Pin_1), J7.5 (Pin_5), U5.1 (OUT)
Other:
- note added: "Na PCB, certifique-se de que o pad de cobre central (sob o componente) esteja conectado ao plano de terra interno por meio de pelo menos uma "via" térmica (thermal via), se possível, ou diretamente ao plano de terra da camada superior."
- moved on the sheet: C19, C20, C21, C22, C23, C24, C25, C26, FB1, J2, J3, J4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

Commit message: Muitas mudanças no circuito, clocks no stm32h7 e mais,
Parts:
- removed D1: APA102-2020, LED_SMD:LED-APA102-2020, symbol LED:APA102-2020
- removed JP1: ID_WP, symbol Jumper:SolderJumper_2_Open
- removed SW1: SW_MEC_5G, Button_Switch_SMD:SW_MEC_5GSH9, symbol Switch:SW_MEC_5G
- removed U2: STM32H753VITx, Package_QFP:LQFP-100_14x14mm_P0.5mm, symbol MCU_ST_STM32H7:STM32H753VITx
- removed U3: TPS7A4700RGWR, TPS7A4700RGWR:QFN65P500X500X100-21N, symbol TPS7A4700:TPS7A4700RGWR
- added C34: 10μF, symbol Device:C_Polarized
- added C35, C52: 1μF, symbol Device:C_Small
- added C36, C54, C55: 100ηF, symbol Device:C_Small
- added C37: 2.2μF X7R 10V, symbol Device:C_Small
- added C38, C39, C40, C41, C42, C43, C44, C45, C46, C47, C48: 100ƞF, symbol Device:C_Small
- added C49: 4.7μF, symbol Device:C_Small
- added C50, C51: 2.2μF, symbol Device:C_Small
- added C53: 10ηF, symbol Device:C_Small
- added C56, C57: 15pF, 0603C, symbol *:root_3_CAP_*_0
- added C58, C59: 15pF, 0603C, symbol MCD_TOOLS:root_2_Capacitor_ST_MCD_TOOLS.SchLib
- added F1: PTC MF-RG300, symbol Device:Polyfuse_Small
- added FB3, FB4: 600 Ω SMD, symbol Device:FerriteBead_Small
- added JP1: Gravação, symbol Jumper:Jumper_2_Small_Open
- added R15, R16, R17, R18: 47R, symbol Device:R_Small
- added R19: 10k, symbol Device:R_Small
- added R20, R21, R22, R23: 100R, symbol Device:R_Small
- added U3: TPS7A2033DQN, Package_SON:Texas_X2SON-4_1x1mm_P0.65mm, symbol Regulator_Linear:TPS7A20xxxDQN
- added U6: STM32H753ZITx, Package_QFP:LQFP-144_20x20mm_P0.5mm, symbol MCU_ST_STM32H7:STM32H753ZITx
- added X1: NX3225HA-25MHz-EXS00A-CH00343, XTAL_4SM_3R2X2R5, symbol MB1246:root_0_NX3225HA-25MHz-EXS00A-CH00343_MB1246.SCHLIB
- added X2: NX3215SA-32.768KHZ-EXS00A-MU00525, XTAL_2SM_3R2X1R5, symbol MB1167:root_1_CRYSTAL_32K_MB1167.SCHLIB_0
Connections:
- net +3V3: now also R19.1
- net +5V: now also F1.1, FB3.2; no longer J1.2 (Pin_2), J1.4 (Pin_4)
- net EN_LEFT: now also U3.3 (EN), U6.58 (PE7)
- net EN_RIGHT: now also U6.59 (PE8)
- net GND: now also U1.1 (A0), U1.2 (A1), U1.3 (A2), C34.2, C35.2, C36.2, C37.2, C38.1, C39.1, C40.1, C41.1, C42.1, C43.1, C44.1, C45.1, C46.1, C47.1, C48.1, C49.2, C50.2, C51.2, C52.2, C53.2, C54.2, C55.2, C56.2, C57.2, C58.2, C59.2, JP1.2 (B), U3.2 (GND), U3.5 (Pad), U6.107 (VSS), U6.120 (VSS), U6.130 (VSS), U6.16 (VSS), U6.38 (VSS), U6.51 (VSS), U6.61 (VSS), U6.83 (VSS), U6.94 (VSS), X1.2, X1.4
- net PDM_CLOCK: now also R15.1
- net PDM_DATA0: now also R17.2
- net PDM_DATA1: now also R18.2
- net PDM_DATA2: now also R16.2
- net at U1.7 (WP): now also JP1.1 (A), R19.2
- new net: F1.2, J1.2 (Pin_2), J1.4 (Pin_4)
- new net: C59.1, R23.2, X2.1
- new net: C58.1, R22.2, X2.2
- new net: C57.1, R21.1, X1.1
- new net: R21.2, U6.24 (PH1)
- new net: C56.1, R20.1, X1.3
- new net: C50.1, U6.71 (VCAP)
- new net: C34.1, C35.1, C36.1, FB3.1, U3.4 (IN)
- new net: R20.2, U6.23 (PH0)
- new net: R17.1, U6.27 (PC1)
- new net: C51.1, U6.106 (VCAP)
- new net: C55.1, FB4.2, U6.33 (VDDA)
- new net: R16.1, U6.45 (PC5)
- new net: R18.1, U6.47 (PB1)
- new net: R15.2, U6.60 (PE9)
- new net: R23.1, U6.8 (PC14)
- new net: R22.1, U6.9 (PC15)
- new net VDD_STM_3.3: C37.1, C38.2, C39.2, C40.2, C41.2, C42.2, C43.2, C44.2, C45.2, C46.2, C47.2, C48.2, C49.1, C52.1, C53.1, C54.1, FB4.1, U3.1 (OUT), U6.108 (VDD), U6.121 (VDD), U6.131 (VDD), U6.143 (PDR_ON), U6.144 (VDD), U6.17 (VDD), U6.30 (VDD), U6.39 (VDD), U6.52 (VDD), U6.62 (VDD), U6.72 (VDD), U6.84 (VDD), U6.95 (VDD33_USB)
- no-connect marks 3 -> 0
Other:
- note added: "Coloque o capacitor de 4.7UF (C49) equidistante aos pinos."
- note added: "Como o PC3_C e o PC2_C estão localizados em uma área do chip cercada por pinos de alimentação analógica (VDDA, VREF+), tome cuidado extra no roteamento: Mantenha a trilha digital do PDM_DATA0 o mais curta possível nessa região. Evite que essa trilha digital cruze ou corra paralelamente a trilhas de referências analógicas sensíveis, para não injetar ruído digital no domínio analógico do microcontr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"
- note added: "Como o pino 60 (Clock) está imprensado entre trilhas de alimentação, certifique-se de que o plano de terra na camada interna seja contínuo sob essa área. Isso impedirá que o ruído digital do clock contamine os trilhos de energia limpa que projetamos."
- note added: "ID_SD and ID_SC PINS: These pins are reserved for HAT ID EEPROM. Lembre-se 100nF muito próximo do chip. O mais próximo possível."
- note added: "No reference design usam 3.2pf, mas no cálculo cheguei a no mínimo 12pf."
- note added: "Não esqueça de configurar o pino PE9 no código do STM32 com High Speed / High Drive Strength para garantir que as bordas do clock permaneçam nítidas para todos os microfones."
- note added: "Resumo das conexões TPS7A2033DQN] Pino, Nome, Conexão 1, OUT, Saída 3.3 V → VDD_LEFT_3.3 (com C26 próximo) 2, NC, Deixar flutuando (não conectar) 3, EN, Conectar a VDD_IN (5 V) ou a OUT (3.3 V) 4, IN, Entrada de VDD_IN (após FB1 e caps de entrada) 5, GND, Conectar ao GND (plano sólido) 6-10, GND/NC, Todos os GND ao plano; NC flutuando Pad, Thermal Pad, Soldar ao GND com múltiplas vias térmicas"
- note removed: "Additional pin functions: https://pinout.xyz/"
- note removed: "ID_SD and ID_SC PINS: These pins are reserved for HAT ID EEPROM. At boot time this I2C interface will be interrogated to look for an EEPROM that identifes the attached board and allows automagic setup of the GPIOs (and optionally, Linux drivers). Bridging JP1 enables write protection. DO NOT USE these pins for anything other than attaching an I2C ID EEPROM. Leave unconnected if ID EEPROM not requ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"
- moved on the sheet: C19, C20, C21, C22, C23, C24, C25, C26, C27, C28, C29, C30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

Commit message: correções, VDD, VSS e outros pinos relevantes para contexto.
 ### Decoupling Strategy for STM32H753 Power Pins

 The STM32H753 microcontroller is a high-performance Cortex-M7 device operating at up to 480 MHz, with integrated USB High-Speed functionality. Such high-speed operation demands a robust power supply decoupling strategy to ensure signal integrity and minimize electromagnetic interference (EMI). Below is the detailed decoupling approach implemented in the AuralFocus HAT design:

 **1. Global Power Filtering**
 - **Ferrite Bead (FB3 - 600 Ω @ 100 MHz)**: placed on the main 3.3 V supply line feeding the STM32H753. This ferrite bead attenuates high-frequency noise originating from upstream sources (e.g., Raspberry Pi power supply, servo motors) before it reaches the microcontroller.
 - **Post-Ferrite Capacitor Bank**:
Parts:
- added C60, C63: 100nF, symbol Device:C_Small
- added C61: 100ηF, symbol Device:C_Small
- added C62: 1μF, symbol Device:C_Small
- added C64, C65: 22μF, symbol Device:C_Small
- added FB5: 600 Ω SMD, symbol Device:FerriteBead_Small
- X2: value NX3215SA-32.768KHZ-EXS00A-MU00525 -> NX3215SA-32.768KHZ; Value2 (none) -> -EXS00A-MU00525
Connections:
- net +5V: now also U3.3 (EN)
- net EN_LEFT: no longer U3.3 (EN), U5.3 (EN)
- net EN_RIGHT: now also U5.3 (EN)
- net GND: now also U6.31 (VSSA), C60.2, C61.2, C62.2, C63.2, C64.2, C65.2
- net VDD_STM_3.3: now also U6.6 (VBAT), C61.1, C63.1, C64.1, FB5.2
- net at C50.1, U6.71 (VCAP): now also C51.1, U6.106 (VCAP), C60.1, C65.1
- net at U6.32 (VREF+): now also C62.1, FB5.1
Other:
- note added: "C64 e c65 devem ficar longe dos LDOs"
- note added: "Não misturar o VSSA com o plano de terra digital em múltiplos locais. Conecte o pino 31 ao terra principal da placa em apenas um ponto físico, preferencialmente sob o microcontrolador."
- moved on the sheet: C37, C38, C39, C40, C41, C42, C43, C44, C45, C46, C47, C48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

Commit message: inclusão dos datasheets e dos circuitos de usb, para alimentação dos servos e para o audio
Parts:
- added C66, C71: 100ηF, symbol Device:C_Small
- added C67, C70: 10μF, symbol Device:C_Small
- added C68: 4.7nF, symbol Device:C_Small
- added C72: 1000μF, symbol Device:C_Small
- added CR1: SMBJ5.0A-TR, SMB_STM, symbol 2026-01-05_21-14-23:SMBJ5.0A-TR
- added FB6: 600 Ω SMD, symbol Device:FerriteBead_Small
- added FB7: 600 Ω 3/4A, symbol Device:FerriteBead_Small
- added J8: USB_C_Receptacle_AUDIO, symbol Connector:USB_C_Receptacle_USB2.0_14P
- added J9: USB_C_Receptacle_SERVOS_POWER, symbol Connector:USB_C_Receptacle_USB2.0_14P
- added R24, R25, R26, R27, R28: 33R, symbol Device:R_Small
- added R29, R30, R34, R35: 5K1, symbol Device:R_Small
- added R31: 1M, symbol Device:R_Small
- added R32: 10k, symbol Device:R_Small
- added R33: 15k, symbol Device:R_Small
- added U2: USBLC6-2SC6, Package_TO_SOT_SMD:SOT-23-6, symbol Power_Protection:USBLC6-2SC6
Connections:
- net PDM_CLOCK is gone; now on net GND: J2.3 (Pin_3), J3.3 (Pin_3), J4.3 (Pin_3), J5.3 (Pin_3), J6.3 (Pin_3), J7.3 (Pin_3), R15.1
- net PDM_DATA1 is gone; now on net GND: J3.4 (Pin_4), J6.4 (Pin_4), R18.2
- net VDD_LEFT_3.3 is gone; now on net GND: C19.1, C20.1, C21.1, C26.1, J2.1 (Pin_1), J3.1 (Pin_1), J4.1 (Pin_1), U4.1 (OUT)
- net GND: now also C66.2, C67.2, C68.2, C70.2, C72.2, J8.A1 (GND), J8.A12 (GND), J8.B1 (GND), J8.B12 (GND), R29.1, R30.1, R31.1, R33.2, U2.2 (GND)
- net GPIO10/SPI0.MOSI: now also R28.2
- net GPIO11/SPI0.SCLK: now also R26.2
- net GPIO24: now also R24.2
- net GPIO8/SPI0.CE0: now also R25.2
- net GPIO9/SPI0.MISO: now also R27.2
- net AUDIO_VBUS: now reaches U6.101 (USB_OTG_FS_VBUS_PA9)
- net AUDIO_VBUS: now also R32.2, R33.1
- net USBD-: now reaches U6.103 (USB_D-_PA11)
- net USBD-: now also U2.6 (I/O1)
- net USBD+: now reaches U6.104 (USB_D+_PA12)
- net USBD+: now also U2.4 (I/O2)
- net at U6.37 (GPIO_Output_PA3): now also R24.1
- net at U6.40 (SPI1_NSS_PA4): now also R25.1
- net at U6.41 (SPI1_SCK_PA5): now also R26.1
- net at U6.42 (SPI1_MISO_PA6): now also R27.1
- net at U6.43 (SPI1_MOSI_PA7): now also R28.1
- new net: J8.A5 (CC1), R29.2
- new net: J8.A7 (D-), J8.B7 (D-), U2.1 (I/O1)
- new net: J8.A6 (D+), J8.B6 (D+), U2.3 (I/O2)
- new net: C66.1, FB6.1, R32.1, U2.5 (VBUS)
- new net: C68.1, J8.S1 (SHIELD), R31.2
- new net: C67.1, FB6.2, J8.A4 (VBUS), J8.A9 (VBUS), J8.B4 (VBUS), J8.B9 (VBUS)
- new net: J8.B5 (CC2), R30.2
- new net: C72.1, CR1.1, FB7.2, J9.A4 (VBUS), J9.A9 (VBUS), J9.B4 (VBUS), J9.B9 (VBUS)
- new net: J9.A5 (CC1), R34.2
- new net: J9.B5 (CC2), R35.2
- new net GND_SERVO: C71.2, CR1.2, J9.A1 (GND), J9.A12 (GND), J9.B1 (GND), J9.B12 (GND), J9.S1 (SHIELD), R34.1, R35.1
- new net V_SERVO_IN: C70.1, C71.1, FB7.1
Other:
- note added: "Este capacitor deve ficar o mais próximo possível dos pino 5 e 2 do USBLC6-2sc6"
- note added: "Faça com que o terra do USB-C de áudio seja sólido com o terra digital do STM32."
- note added: "Isolar o GND e o V_SERVO Para retirar o ruido dos motores do barramento de controle digital"
- note added: "Mantenha o ponto de união (Net Tie ou Star Ground) entre o GND_SERVO e o GND_DIGITAL em um local estratégico, geralmente próximo à entrada principal de energia ou ao regulador de tensão,"
- note added: "Os pinos B9, A9, B4 estão invisíveis e são VBUS Os pinos A12, B1, B12 estão invisíveis e são GND"
- note added: "rotear as trilhas USB D- e D+ como um par diferencial com impedância de 90Ω"
- moved on the sheet: C19, C20, C21, C22, C23, C24, C25, C26, C27, C28, C29, C30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
